File: hardware/schematics/the-SAD.kicad_sch (KiCad schematic)
At the start: 5 parts, among them M1 Motor_DC, U2 DHT22

Commit message: forgot to add the led
Parts:
- added D1: LED, symbol Device:LED
- added R1: 220Ω, symbol Device:R
Connections:
- net at A1.21 (D6): now also R1.2
- net at A1.7 (GND): now also D1.1 (K)
- new net: D1.2 (A), R1.1
Other:
- note added: "Crank LED"
Changed lines of the file:
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@@
+		)
+	)
+	(text "Crank LED"
+		(exclude_from_sim no)
+		(at 54.864 85.344 0)
+		(effects
+			(font
+				(size 1.778 1.778)
+			)
 		)
 	)
@@
 	(wire
 		(pts
+			(xy 104.14 88.9) (xy 104.14 43.18)
+		)
+		(stroke
+			(width 0)
+			(type default)
+			(color 255 174 67 1)
+		)
+	)
+	(wire
+		(pts
+			(xy 64.77 81.28) (xy 109.22 81.28)
+		)
+		(stroke
+			(width 0)
+			(type default)
+			(color 0 0 0 1)
+		)
+	)
+	(wire
+		(pts
+			(xy 109.22 81.28) (xy 109.22 68.58)
+		)
+		(stroke
+			(width 0)
+			(type default)
+			(color 0 0 0 1)
+		)
+	)
+	(wire
+		(pts
 			(xy 64.77 63.5) (xy 85.09 63.5)
 		)
@@
 	(wire
 		(pts
+			(xy 137.16 43.18) (xy 137.16 53.34)
+		)
+		(stroke
+			(width 0)
+			(type default)
+			(color 255 174 67 1)
+		)
+	)
+	(wire
+		(pts
 			(xy 85.09 45.72) (xy 85.09 50.8)
 		)
@@
 	(wire
 		(pts
+			(xy 64.77 88.9) (xy 72.39 88.9)
+		)
+		(stroke
+			(width 0)
+			(type default)
+			(color 255 174 67 1)
+		)
+	)
+	(wire
+		(pts
 			(xy 95.25 38.1) (xy 147.32 38.1)
 		)
@@
 	(wire
 		(pts
+			(xy 104.14 43.18) (xy 137.16 43.18)
+		)
+		(stroke
+			(width 0)
+			(type default)
+			(color 255 174 67 1)
+		)
+	)
+	(wire
+		(pts
 			(xy 85.09 63.5) (xy 85.09 66.04)
 		)
@@
 	(wire
 		(pts
+			(xy 80.01 88.9) (xy 104.14 88.9)
+		)
+		(stroke
+			(width 0)
+			(type default)
+			(color 255 174 67 1)
+		)
+	)
+	(wire
+		(pts
 			(xy 173.99 45.72) (xy 129.54 45.72)
 		)
@@
 			(type default)
 			(color 0 0 0 1)
+		)
+	)
+	(symbol
+		(lib_id "Device:R")
+		(at 76.2 88.9 90)
+		(unit 1)
+		(exclude_from_sim no)
+		(in_bom yes)
+		(on_board yes)
+		(dnp no)
+		(property "Reference" "R1"
+			(at 76.2 83.566 90)
+			(effects
+				(font
+					(size 1.27 1.27)
+				)
+			)
+		)
+		(property "Value" "220Ω"
+			(at 76.2 86.106 90)
+			(effects
+				(font
+					(size 1.27 1.27)
+				)
+			)
+		)
+		(property "Footprint" ""
+			(at 76.2 90.678 90)
+			(effects
+				(font
+					(size 1.27 1.27)
+				)
+				(hide yes)
+			)
+		)
+		(property "Datasheet" "~"
+			(at 76.2 88.9 0)
+			(effects
+				(font
+					(size 1.27 1.27)
+				)
+				(hide yes)
+			)
+		)
+		(property "Description" "Resistor"
+			(at 76.2 88.9 0)
+			(effects
+				(font
+					(size 1.27 1.27)
+				)
+				(hide yes)
+			)
+		)
+		(pin "2"
+		)
+		(pin "1"
+		)
+		(instances
+			(project ""
+				(path "/39c0e1e3-ef71-415d-b89e-994d0ea5b8e0"
+					(reference "R1")
+					(unit 1)
+				)
+			)
 		)
 	)
@@
 					(unit 1)
 				)
+			)
+		)
+	)
+	(symbol
+		(lib_id "Device:LED")
+		(at 64.77 85.09 270)
+		(unit 1)
+		(exclude_from_sim no)
+		(in_bom yes)
+		(on_board yes)
+		(dnp no)
+		(property "Reference" "D1"
+			(at 67.31 83.82 90)
+			(effects
+				(font
+					(size 1.27 1.27)
+				)
+				(justify left)
+			)
+		)
+		(property "Value" "LED"
+			(at 67.31 86.36 90)
+			(effects
+				(font
+					(size 1.27 1.27)
+				)
+				(justify left)
+			)
+		)
+		(property "Footprint" ""
+			(at 64.77 85.09 0)
+			(effects
+				(font
+					(size 1.27 1.27)
+				)
+				(hide yes)
+			)
+		)
+		(property "Datasheet" "~"
+			(at 64.77 85.09 0)
+			(effects
+				(font
+					(size 1.27 1.27)
+				)
+				(hide yes)
+			)
+		)
+		(property "Description" "Light emitting diode"
+			(at 64.77 85.09 0)
+			(effects
+				(font
+					(size 1.27 1.27)
+				)
+				(hide yes)
+			)
+		)
+		(property "Sim.Pins" "1=K 2=A"
+			(at 64.77 85.09 0)
+			(effects
+				(font
+					(size 1.27 1.27)
+				)
+				(hide yes)
+			)
+		)
+		(pin "1"
+		)
+		(pin "2"
+		)
+		(instances
+			(project ""
+				(path "/39c0e1e3-ef71-415d-b89e-994d0ea5b8e0"
+					(reference "D1")
+					(unit 1)
+				)
